File: project/_input3.kicad_sch (KiCad schematic)
At the start: 19 parts, among them J7 input_1x5, U8 LTV-244-GB-G

Commit message: bom fixes
Parts:
- R70, R71, R72, R73, R74, R75, R76, R77: lcsc# (none) -> C17379
Changed lines of the file:
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@@
       (effects (font (size 1.27 1.27)) hide)
     )
-    (property "lcsc#" "" (id 5) (at 132.08 109.22 0)
+    (property "lcsc#" "C17379" (id 5) (at 132.08 109.22 0)
       (effects (font (size 1.27 1.27)) hide)
     )
@@
       (effects (font (size 1.27 1.27)) hide)
     )
-    (property "lcsc#" "" (id 5) (at 124.46 33.02 0)
+    (property "lcsc#" "C17379" (id 5) (at 124.46 33.02 0)
       (effects (font (size 1.27 1.27)) hide)
     )
@@
       (effects (font (size 1.27 1.27)) hide)
     )
-    (property "lcsc#" "" (id 5) (at 124.46 109.22 0)
+    (property "lcsc#" "C17379" (id 5) (at 124.46 109.22 0)
       (effects (font (size 1.27 1.27)) hide)
     )
@@
       (effects (font (size 1.27 1.27)) hide)
     )
-    (property "lcsc#" "" (id 5) (at 124.46 147.32 0)
+    (property "lcsc#" "C17379" (id 5) (at 124.46 147.32 0)
       (effects (font (size 1.27 1.27)) hide)
     )
@@
       (effects (font (size 1.27 1.27)) hide)
     )
-    (property "lcsc#" "" (id 5) (at 132.08 71.12 0)
+    (property "lcsc#" "C17379" (id 5) (at 132.08 71.12 0)
       (effects (font (size 1.27 1.27)) hide)
     )
@@
       (effects (font (size 1.27 1.27)) hide)
     )
-    (property "lcsc#" "" (id 5) (at 132.08 33.02 0)
+    (property "lcsc#" "C17379" (id 5) (at 132.08 33.02 0)
       (effects (font (size 1.27 1.27)) hide)
     )
@@
       (effects (font (size 1.27 1.27)) hide)
     )
-    (property "lcsc#" "" (id 5) (at 124.46 71.12 0)
+    (property "lcsc#" "C17379" (id 5) (at 124.46 71.12 0)
       (effects (font (size 1.27 1.27)) hide)
     )
@@
       (effects (font (size 1.27 1.27)) hide)
     )
-    (property "lcsc#" "" (id 5) (at 132.08 147.32 0)
-      (effects (font (size 1.27 1.27)) hide)
-    )
+    (property "lcsc#" "C17379" (id 5) (at 132.08 147.32 0)
+      (effects (font (size 1.27 1.27)) hide)
+    )
